File: connectors.kicad_sch (KiCad schematic)
At the start: 0 parts

Commit message: assigned footprint libraries
Parts:
- added J1, J2: Conn_01x04_Pin, Connector_PinHeader_2.54mm:PinHeader_1x04_P2.54mm_Vertical, symbol Connector:Conn_01x04_Pin
- added J3: Conn_01x09_Pin, Connector_PinHeader_2.54mm:PinHeader_1x09_P2.54mm_Vertical, symbol Connector:Conn_01x09_Pin
- added J4: Conn_02x03_Odd_Even, Connector_PinHeader_2.54mm:PinHeader_2x03_P2.54mm_Vertical, symbol Connector_Generic:Conn_02x03_Odd_Even

Commit message: finished project
Connections:
- net GND: now reaches J2.1 (Pin_1)
- net GND: now also J1.1 (Pin_1), J3.8 (Pin_8), J4.6 (Pin_6)
- net Vcc: now reaches J2.2 (Pin_2)
- net Vcc: now also J1.2 (Pin_2), J3.9 (Pin_9), J4.2 (Pin_2)
- net RX: now reaches J2.3 (Pin_3)
- net TX: now reaches J2.4 (Pin_4)
- net D2: now reaches J3.1 (Pin_1)
- net D3: now reaches J3.2 (Pin_2)
- net D4: now reaches J3.3 (Pin_3)
- net D5: now reaches J3.4 (Pin_4)
- net D6: now reaches J3.5 (Pin_5)
- net D7: now reaches J3.6 (Pin_6)
- net D8: now reaches J3.7 (Pin_7)
- net SDA: now reaches J1.3 (Pin_3)
- net SCL: now reaches J1.4 (Pin_4)
- net SCL: now also J4.3 (Pin_3)
- net MISO: now reaches J4.1 (Pin_1)
- net MOSI: now reaches J4.4 (Pin_4)
- net RESET: now reaches J4.5 (Pin_5)
